File: PSU.kicad_pcb (KiCad board)
At the start: 2 copper layers, 91.4 x 105.4 mm, 68 parts, among them J1 +12V in1, J10 +5V, J11 0V, J2 +12V in2, J3 0v, J4 Conn_02x20_Odd_Even, J5 LED-, J6 LED+, J7 Sw, J8 Sw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

Commit message: Updates prior to pcb order.
Parts:
- J1, J10, J11, J2, J3, J9: footprint my_extras:SolderConnector -> my_extras:SolderConnector - HighCurrent
- moved C11 1.91 mm to (165.1, 88.3)
Routing:
- net Net-(C11-Pad1): track 68.4 -> 70.1 mm
- net Net-(C1-Pad1): track 209.7 -> 210.8 mm
- net GND: track 88.7 -> 89.7 mm
- net Net-(C6-Pad2): track 78.3 -> 77.6 mm
Other:
- board text added: "+5V"
- board text added: "+5Vu"
- board text added: "0V"
- board text added: "12V in1"
- board text added: "12V in2"
- board text added: "Graceful-Shutdown 12V Rpi Power Supply"
- board text added: "LED+"
- board text added: "LED-"
- board text added: "Sw"
- board text added: "https://github.com/marcmunro/GracefulPSU"
- board text added: "https://github.com/marcmunro/GracefulPSU.git"
