File: PSU.kicad_sch (KiCad schematic)
At the start: 60 parts, among them J1 +12V in1, J10 +5V, J11 0V, J2 +12V in2, J3 0v, J4 Conn_02x20_Odd_Even, J5 LED-, J6 LED+, J7 Sw, J8 Sw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

Commit message: Prep for release to github
Parts:
- Q2: footprint my_extras:SOIC127P600X175-8N -> SOIC127P600X175-8N
Changed lines of the file:
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@@
       (effects (font (size 1.27 1.27)) (justify left))
     )
-    (property "Footprint" "my_extras:SOIC127P600X175-8N" (id 2) (at 151.13 104.14 0)
+    (property "Footprint" "SOIC127P600X175-8N" (id 2) (at 151.13 104.14 0)
       (effects (font (size 1.27 1.27)) (justify left bottom) hide)
     )
@@
     (property "Reference" "Q2" (id 0) (at 154.94 63.5 90))
     (property "Value" "IRF7319" (id 1) (at 153.67 55.2474 90))
-    (property "Footprint" "my_extras:SOIC127P600X175-8N" (id 2) (at 153.67 58.42 0)
+    (property "Footprint" "SOIC127P600X175-8N" (id 2) (at 153.67 58.42 0)
       (effects (font (size 1.27 1.27)) (justify left bottom) hide)
     )
@@
     )
     (path "/8313aa4b-6cbb-4625-849b-7a8ca7be5fa2"
-      (reference "Q2") (unit 1) (value "IRF7319") (footprint "my_extras:SOIC127P600X175-8N")
+      (reference "Q2") (unit 1) (value "IRF7319") (footprint "SOIC127P600X175-8N")
     )
     (path "/a5e7c297-8404-4078-b7f8-933e1625a329"
-      (reference "Q2") (unit 2) (value "IRF7319") (footprint "my_extras:SOIC127P600X175-8N")
+      (reference "Q2") (unit 2) (value "IRF7319") (footprint "SOIC127P600X175-8N")
     )
     (path "/3cdf56f1-911a-4c7d-85ba-496fd2ca049d"

Commit message: Updates prior to pcb order.
Parts:
- J1, J10, J11, J2, J3, J9: footprint my_extras:SolderConnector -> my_extras:SolderConnector - HighCurrent
- Q2: footprint SOIC127P600X175-8N -> my_extras:SOIC127P600X175-8N
Changed lines of the file:
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@@
       (effects (font (size 1.27 1.27)) (justify left))
     )
-    (property "Footprint" "my_extras:SolderConnector" (id 2) (at 259.08 86.36 0)
+    (property "Footprint" "my_extras:SolderConnector - HighCurrent" (id 2) (at 259.08 86.36 0)
       (effects (font (size 1.27 1.27)) hide)
     )
@@
       (effects (font (size 1.27 1.27)) (justify left))
     )
-    (property "Footprint" "SOIC127P600X175-8N" (id 2) (at 151.13 104.14 0)
+    (property "Footprint" "my_extras:SOIC127P600X175-8N" (id 2) (at 151.13 104.14 0)
       (effects (font (size 1.27 1.27)) (justify left bottom) hide)
     )
@@
     (property "Reference" "Q2" (id 0) (at 154.94 63.5 90))
     (property "Value" "IRF7319" (id 1) (at 153.67 55.2474 90))
-    (property "Footprint" "SOIC127P600X175-8N" (id 2) (at 153.67 58.42 0)
+    (property "Footprint" "my_extras:SOIC127P600X175-8N" (id 2) (at 153.67 58.42 0)
       (effects (font (size 1.27 1.27)) (justify left bottom) hide)
     )
@@
       (effects (font (size 1.27 1.27)) (justify left))
     )
-    (property "Footprint" "my_extras:SolderConnector" (id 2) (at 259.08 114.3 0)
+    (property "Footprint" "my_extras:SolderConnector - HighCurrent" (id 2) (at 259.08 114.3 0)
       (effects (font (size 1.27 1.27)) hide)
     )
@@
     (property "Reference" "J3" (id 0) (at 17.145 103.5263 0))
     (property "Value" "0v" (id 1) (at 17.145 112.6514 0))
-    (property "Footprint" "my_extras:SolderConnector" (id 2) (at 16.51 114.3 0)
+    (property "Footprint" "my_extras:SolderConnector - HighCurrent" (id 2) (at 16.51 114.3 0)
       (effects (font (size 1.27 1.27)) hide)
     )
@@
     (property "Reference" "J2" (id 0) (at 17.145 33.6763 0))
     (property "Value" "+12V in2" (id 1) (at 17.145 36.4514 0))
-    (property "Footprint" "my_extras:SolderConnector" (id 2) (at 16.51 38.1 0)
+    (property "Footprint" "my_extras:SolderConnector - HighCurrent" (id 2) (at 16.51 38.1 0)
       (effects (font (size 1.27 1.27)) hide)
     )
@@
       (effects (font (size 1.27 1.27)) (justify left))
     )
-    (property "Footprint" "my_extras:SolderConnector" (id 2) (at 259.08 96.52 0)
+    (property "Footprint" "my_extras:SolderConnector - HighCurrent" (id 2) (at 259.08 96.52 0)
       (effects (font (size 1.27 1.27)) hide)
     )
@@
     (property "Reference" "J1" (id 0) (at 17.145 26.0563 0))
     (property "Value" "+12V in1" (id 1) (at 17.145 28.8314 0))
-    (property "Footprint" "my_extras:SolderConnector" (id 2) (at 16.51 30.48 0)
+    (property "Footprint" "my_extras:SolderConnector - HighCurrent" (id 2) (at 16.51 30.48 0)
       (effects (font (size 1.27 1.27)) hide)
     )
@@
     )
     (path "/ee2ac6c1-0f19-4149-8109-f33c6cf39572"
-      (reference "J1") (unit 1) (value "+12V in1") (footprint "my_extras:SolderConnector")
+      (reference "J1") (unit 1) (value "+12V in1") (footprint "my_extras:SolderConnector - HighCurrent")
     )
     (path "/c04483c4-a6e0-4698-9634-11e2a88f9c38"
-      (reference "J2") (unit 1) (value "+12V in2") (footprint "my_extras:SolderConnector")
+      (reference "J2") (unit 1) (value "+12V in2") (footprint "my_extras:SolderConnector - HighCurrent")
     )
     (path "/b8f266dc-1231-4e57-9c4d-fe42c8f637ec"
-      (reference "J3") (unit 1) (value "0v") (footprint "my_extras:SolderConnector")
+      (reference "J3") (unit 1) (value "0v") (footprint "my_extras:SolderConnector - HighCurrent")
     )
     (path "/9654f0de-99cd-4a0b-97ac-04fe683fda27"
@@
     )
     (path "/759c7969-f4bd-434e-81a8-4e70b628dc37"
-      (reference "J9") (unit 1) (value "+5Vu") (footprint "my_extras:SolderConnector")
+      (reference "J9") (unit 1) (value "+5Vu") (footprint "my_extras:SolderConnector - HighCurrent")
     )
     (path "/cf96d0cf-db7b-47c7-8b87-1b01593afa18"
-      (reference "J10") (unit 1) (value "+5V") (footprint "my_extras:SolderConnector")
+      (reference "J10") (unit 1) (value "+5V") (footprint "my_extras:SolderConnector - HighCurrent")
     )
     (path "/b312beb6-cfaa-4682-b995-12f6f2cbbd78"
-      (reference "J11") (unit 1) (value "0V") (footprint "my_extras:SolderConnector")
+      (reference "J11") (unit 1) (value "0V") (footprint "my_extras:SolderConnector - HighCurrent")
     )
     (path "/48d8e6b0-6585-4cd3-9de6-465e1d727e2e"
@@
     )
     (path "/8313aa4b-6cbb-4625-849b-7a8ca7be5fa2"
-      (reference "Q2") (unit 1) (value "IRF7319") (footprint "SOIC127P600X175-8N")
+      (reference "Q2") (unit 1) (value "IRF7319") (footprint "my_extras:SOIC127P600X175-8N")
     )
     (path "/a5e7c297-8404-4078-b7f8-933e1625a329"
-      (reference "Q2") (unit 2) (value "IRF7319") (footprint "SOIC127P600X175-8N")
+      (reference "Q2") (unit 2) (value "IRF7319") (footprint "my_extras:SOIC127P600X175-8N")
     )
     (path "/3cdf56f1-911a-4c7d-85ba-496fd2ca049d"
