File: kicad/PSU.kicad_pcb (KiCad board)
At the start: 2 copper layers, 91.4 x 105.4 mm, 68 parts, among them J1 +12V in1, J10 +5V, J11 0V, J2 +12V in2, J3 0v, J4 Conn_02x20_Odd_Even, J5 LED-, J6 LED+, J7 Sw, J8 Sw, J9 +5Vu, Q1 CSD19505, Q2 IRF7319, Q3 CSD19505KCS, U1 LM358, U2 LM22678TJ-ADJ

Commit message: Still setting up...
Parts:
- removed the C5 at (115.5, 125.7)
- removed the C6 at (115.5, 130.8)
- added C8: 1μF, Capacitor_THT:C_Disc_D7.5mm_W2.5mm_P5.00mm, F.Cu at (102.9, 130.8)
- added C9: 1uF, Capacitor_THT:C_Disc_D7.5mm_W2.5mm_P5.00mm, F.Cu at (110.5, 97.1)
- added D10: 6.8V, Diode_THT:D_A-405_P7.62mm_Horizontal, F.Cu at (137.2, 116.8)
- added D11: D, Diode_THT:D_A-405_P7.62mm_Horizontal, F.Cu at (108.0, 137.2)
- added D9: D, Diode_THT:D_A-405_P7.62mm_Horizontal, F.Cu at (110.5, 160.0)
- added R22: 100K, Resistor_THT:R_Axial_DIN0207_L6.3mm_D2.5mm_P10.16mm_Horizontal, F.Cu at (132.1, 127.0)
- added R24: 1M, Resistor_THT:R_Axial_DIN0207_L6.3mm_D2.5mm_P10.16mm_Horizontal, F.Cu at (124.5, 125.7)
- added R25: 4.7M, Resistor_THT:R_Axial_DIN0207_L6.3mm_D2.5mm_P10.16mm_Horizontal, F.Cu at (102.9, 124.5)
- C1: value 16uF -> 10uF; footprint Capacitor_THT:CP_Axial_L18.0mm_D6.5mm_P25.00mm_Horizontal -> Capacitor_THT:CP_Radial_D5.0mm_P2.00mm
- C7: value 10μF -> 1μF; footprint Capacitor_THT:CP_Radial_D5.0mm_P2.00mm -> Capacitor_THT:C_Disc_D7.5mm_W2.5mm_P5.00mm
- D8: value D -> 6.8V
- Q3: value CSD19505KCS -> CSD19505
- R10: value 10M -> 100K
- R11: value 100K -> 47K
- R13: value 430K -> 10K
- R14: value 560K -> 1M
- R15: value 10M -> 1M
- R16: value 12k -> 1M
- R17: value 10K -> 270K
- R19: value 100K -> 4.7M
- R20: value 100K -> 12k
- R21: value 330K -> 10K
- R3: value 1M -> 2M
- R4: value 2M -> 3.9M
- R6: value 330K -> 270K
- R9: value 560K -> 22M
- moved R14 74.1 mm to (167.6, 99.1), turned to 0 degrees
- moved D8 73.1 mm to (105.4, 177.8), turned to 90 degrees
- moved R15 61.5 mm to (163.8, 105.4), turned to 180 degrees
- moved R13 60.8 mm to (153.7, 100.3), turned to 0 degrees
- moved R16 52.2 mm to (105.4, 154.9), turned to 90 degrees
- moved R19 47.0 mm to (100.3, 154.9), turned to 90 degrees
- moved R11 37.4 mm to (111.8, 153.7), turned to 0 degrees
- moved R7 37.0 mm to (111.8, 172.7), turned to -90 degrees
- moved R20 33.1 mm to (108.0, 103.5), turned to -90 degrees
- moved R8 30.5 mm to (111.8, 148.6), turned to 0 degrees
- moved R3 25.2 mm to (118.1, 172.7), turned to -90 degrees
- moved R21 23.9 mm to (113.3, 113.7), turned to 90 degrees
- moved C1 22.0 mm to (124.5, 162.6), turned to -90 degrees
- moved R9 19.4 mm to (134.6, 143.5), turned to 90 degrees
- moved D3 18.5 mm to (124.5, 170.2)
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- renumbered C8 to C5, C9 to C6, D9 to D12, J11 to J10, J9 to J11, J10 to J9, R22 to R23, R23 to R26
Connections:
- C5 pad 1: Net-(C7-Pad1) -> Net-(C5-Pad1)
- C6 pad 1: Net-(C7-Pad1) -> Net-(C5-Pad1)
- C7 pad 1: Net-(C7-Pad1) -> /A
- C7 pad 2: Net-(C7-Pad2) -> /B
- D8 pad 1: Net-(C6-Pad2) -> Net-(D8-Pad1)
- J7 pad 1: Net-(C6-Pad2) -> Net-(C8-Pad2)
- Q2 pad 2: Net-(C7-Pad2) -> Net-(Q2-Pad2)
- Q2 pad 5: Net-(C7-Pad1) -> Net-(C5-Pad1)
- Q2 pad 6: Net-(C7-Pad1) -> Net-(C5-Pad1)
- R10 pad 1: Net-(R10-Pad1) -> GND
- R10 pad 2: Net-(Q1-Pad1) -> Net-(C3-Pad1)
- R11 pad 1: GND -> Net-(D9-Pad1)
- R11 pad 2: Net-(C3-Pad1) -> Net-(D10-Pad2)
- R12 pad 1: Net-(R12-Pad1) -> Net-(D8-Pad1)
- R12 pad 2: Net-(R12-Pad2) -> Net-(C4-Pad2)
- R13 pad 1: Net-(C1-Pad1) -> Net-(D10-Pad1)
- R13 pad 2: Net-(R13-Pad2) -> Net-(Q1-Pad1)
- R14 pad 1: Net-(R13-Pad2) -> Net-(Q1-Pad1)
- R15 pad 1: Net-(R12-Pad2) -> Net-(C4-Pad2)
- R15 pad 2: Net-(C6-Pad2) -> Net-(R15-Pad2)
- R16 pad 1: Net-(J5-Pad1) -> Net-(C1-Pad1)
- R16 pad 2: Net-(C6-Pad2) -> Net-(R16-Pad2)
- R17 pad 1: Net-(C4-Pad1) -> Net-(R16-Pad2)
- R17 pad 2: /B -> GND
- R18 pad 1: Net-(D8-Pad2) -> Net-(D11-Pad2)
- R19 pad 1: Net-(C4-Pad1) -> Net-(R15-Pad2)
- R19 pad 2: /A -> Net-(C8-Pad2)
- R20 pad 1: Net-(C7-Pad1) -> Net-(J5-Pad1)
- R20 pad 2: Net-(D8-Pad2) -> Net-(C8-Pad2)
- R21 pad 1: Net-(D8-Pad2) -> Net-(C4-Pad1)
- R21 pad 2: Net-(C7-Pad2) -> /B
- R4 pad 2: Net-(R10-Pad1) -> Net-(R4-Pad2)
- R6 pad 2: Net-(R12-Pad1) -> Net-(D8-Pad1)
- R7 pad 1: Net-(R12-Pad1) -> Net-(D8-Pad1)
- R9 pad 1: Net-(R12-Pad1) -> Net-(R4-Pad2)
- R9 pad 2: Net-(C4-Pad2) -> Net-(D10-Pad2)
- U1 pad 1: Net-(C6-Pad2) -> Net-(C8-Pad2)
- U1 pad 2: Net-(R13-Pad2) -> Net-(R16-Pad2)
- U1 pad 3: Net-(R12-Pad2) -> Net-(R15-Pad2)
- U1 pad 5: Net-(R12-Pad1) -> Net-(D8-Pad1)
- U1 pad 6: Net-(R10-Pad1) -> Net-(R4-Pad2)
- U1 pad 7: Net-(Q1-Pad1) -> Net-(D10-Pad2)
- U2 pad 2: Net-(C7-Pad1) -> Net-(C5-Pad1)
Routing:
- net Net-(C5-Pad1): track 0.00 -> 92.3 mm, vias 0 -> 2
- net Net-(R15-Pad2): track 0.00 -> 91.4 mm
- net Net-(C7-Pad1): track 80.4 -> 0.00 mm, vias 1 -> 0
- net Net-(C6-Pad2): track 77.6 -> 0.00 mm
- net Net-(Q1-Pad1): track 78.7 -> 11.4 mm
- net Net-(C8-Pad2): track 0.00 -> 64.2 mm
- net Net-(D8-Pad1): track 0.00 -> 56.9 mm
- net Net-(Q2-Pad2): track 0.00 -> 52.0 mm
- net Net-(R12-Pad1): track 48.7 -> 0.00 mm
- net Net-(D10-Pad2): track 0.00 -> 43.6 mm
- net /A: track 24.7 -> 67.0 mm
- net Net-(R16-Pad2): track 0.00 -> 40.1 mm
- net Net-(R4-Pad2): track 0.00 -> 38.0 mm
- net Net-(C4-Pad2): track 73.8 -> 111.4 mm
- net Net-(R12-Pad2): track 35.7 -> 0.00 mm
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Other:
- board text added: "https://github.com/bloodnok-marine/Graceful_PSU.git"
- board text removed: "https://github.com/marcmunro/GracefulPSU"
- board text removed: "https://github.com/marcmunro/GracefulPSU.git"
