File: kicad/simulation/simulation.kicad_sch (KiCad schematic)
At the start: 21 parts, among them Q1 BC547, U1 OPAMP, U2 OPAMP

Commit message: Documentation updates.  Fix to simualation.
Parts:
- Q1: Spice_Lib_File /home/marc/proj/kicad6/psu/PSU/spice/2N2222.lib -> spice/2N2222.lib
Changed lines of the file:
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@@
       (effects (font (size 1.27 1.27)) hide)
     )
-    (property "Spice_Lib_File" "/home/marc/proj/kicad6/psu/PSU/spice/2N2222.lib" (id 7) (at 118.11 81.28 0)
+    (property "Spice_Lib_File" "spice/2N2222.lib" (id 7) (at 118.11 81.28 0)
       (effects (font (size 1.27 1.27)) hide)
     )

Commit message: Still setting up...
Parts:
- removed Q1: BC547, Package_TO_SOT_THT:TO-92_Inline, symbol Transistor_BJT:BC547
- added C3, C4: 1uF, symbol Device:C
- added C5: 1uF, symbol Device:C_Polarized
- added D4, D6: 6V8, symbol Device:D_Zener
- added D5, D7: D, symbol Device:D
- added Q1: CSD19505KCS, Package_TO_SOT_THT:TO-220-3_Vertical, symbol csd19502q5b:CSD19505KCS
- added Q2: 2N2222, Package_TO_SOT_THT:TO-18-3, symbol Transistor_BJT:BC108
- added Q3: Q_PMOS_DGS, symbol Device:Q_PMOS_DGS
- added Q4: Q_NMOS_DGS, symbol Device:Q_NMOS_DGS
- added R10, R17, R18, R19, R20: 1M, symbol Device:R
- added R14, R15: 100R, symbol Device:R
- added R21: 1k, symbol Device:R
- added R6: 47k, symbol Device:R
- added V2, V3: VDC, symbol Simulation_SPICE:VDC
- C1: value 16uF -> 10uF; Spice_Model 16uF -> 10uF
- C2: value 10000uF -> 1.6F; Spice_Model 10000uF -> 1.6
- R12: renamed from R10; value 430K -> 1M; Spice_Model 430k -> 1meg
- R13: renamed from R11; value 560K -> 270K; Spice_Model 560k -> 270k
- R16: renamed from R12; value 10M -> 4.7M; Spice_Model 10Meg -> 4.7Meg
- R2: value 1M -> 2.7M; Spice_Model 1Meg -> 2.7Meg
- R3: value 2M -> 4M; Spice_Model 2Meg -> 4Meg
- R4: value 330k -> 270K; Spice_Model 330k -> 270k
- R7: renamed from R6; value 10M -> 22M; Spice_Model 10Meg -> 22Meg
- R8: renamed from R7; value 560k -> 1M; Spice_Model 560k -> 1meg
- R9: value 1k -> 10k; Spice_Model 1k -> 10k
- V1: Spice_Model dc 12 pulse(0 12 5m 1m 1m 20 60) -> dc 12 pulse(0 12 5m 1m 1m 15 30)
- renumbered R8 to R11
Connections:
- net GND: now also Q1.3 (S), Q2.1 (E), Q4.3 (S), R10.2, R21.2, V2.2, V3.2
- net Vc1: now also D4.1 (K)
- net Vc2: now also R11.1, Q1.2 (D)
- net Vcc: now also Q3.3 (S), R17.1
- net Vgate: now also D6.2 (A), R6.2; no longer R9.1
- net Vin: now also D1.2 (A), D3.2 (A), V1.1; no longer R11.1, R4.2, R5.1, R8.1, U1.1 (+)
- net Vsw: now also C4.1
- net Vcomp0: now reaches R3.2, R7.1, U1.2 (-)
- net Vcomp2: now reaches R12.2, R13.1, U2.2 (-)
- net at R9.2: now also Q1.1 (G), R10.1
- net Vcomp3: now reaches R11.2, R16.1, U2.1 (+)
- new net: Q2.2 (B), R14.2, R15.2
- new net: C5.2, R19.2, R20.1
- new net: C3.2, C4.2, Q3.2 (G), Q4.1 (D), R17.2
- new net: D6.1 (K), R9.1
- new net: D7.2 (A), R18.2, R19.1
- new net: D5.1 (K), R6.1
- new net: D4.2 (A), D5.2 (A)
- new net V2: R14.1, V2.1
- new net V3: R15.1, V3.1
- new net Vcomp1: R4.2, R5.1, R8.1, U1.1 (+)
- new net Vg3: Q4.2 (G), R20.2
- new net Vout: C5.1, Q3.1 (D), R18.1, R21.1
- new net Vq2: C3.1, D7.1 (K), Q2.3 (C)
Other:
- note added: ".tran 1m 70s"
- note added: "Emulation of momentary push for power-on"
- note added: "Emulation of push and hold for power-off"
- note removed: ".tran 1m 100s"
- moved on the sheet: C1, C2, D1, D2, D3, R11, R12, R13, R16, R2, R3, R4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
